File: dcdc_reg.kicad_sch (KiCad schematic)
At the start: 26 parts, among them M1 30V 22A, M2 30V 22A, U9 LM25117PMHX/NOPB

Commit message: Revise following review 1
Parts:
- U9: footprint Package_SO:Texas_PWP0020A -> PWP0020A_N
Changed lines of the file:
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@@
 			)
 		)
-		(property "Footprint" "Package_SO:Texas_PWP0020A"
+		(property "Footprint" "PWP0020A_N"
 			(at 151.13 97.79 0)
 			(effects
