File: motor_driver.kicad_sch (KiCad schematic)
At the start: 7 parts, among them U4 DRV8873SPWPRQ1

Commit message: Revise following review 1
Parts:
- U4: footprint DRV8873:IC_DRV8873SPWPRQ1 -> DRV8873SPWPRQ1:IC_DRV8873SPWPRQ1
Changed lines of the file:
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@@
 			)
 		)
-		(property "Footprint" "DRV8873:IC_DRV8873SPWPRQ1"
+		(property "Footprint" "DRV8873SPWPRQ1:IC_DRV8873SPWPRQ1"
 			(at 128.27 105.41 0)
 			(effects
