File: robot.kicad_sch (KiCad schematic)
At the start: 50 parts, among them J1 Conn_ARM_JTAG_SWD_10, J2 JTAG 5 Pin Custom, J3 MOT1_OUT, J4 MOT2_OUT, J5 XT60-BATT, J6 MOT3_OUT, J7 MOT4_OUT, SW1 Reset, SW2 SW_SPDT, U1 STLINK-V3MODS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

Commit message: Add dip switch, buttons, leds, indiv mot fault pins
Parts:
- added D4: LED_RED, symbol Device:LED
- added D5: LED_BLUE, symbol Device:LED
- added D6: LED_GREEN, symbol Device:LED
- added R37, R38, R39: 1k, symbol Device:R_US
- added R40, R41, R42, R43: 3k3, symbol Device:R_US
- added R44, R45, R46, R47, R48, R49: 10k, symbol Device:R_US
- added SW3: SW_DIP_x04, symbol Switch:SW_DIP_x04
- added SW4, SW5, SW6: SW_SPDT, Button_Switch_THT:SW_PUSH-12mm, symbol Switch:SW_SPDT
Connections:
- net +3.3V: now also R40.1, R41.1, R42.1, R43.1, R44.2, R45.2, R46.2, SW4.1 (A), SW5.1 (A), SW6.1 (A)
- net GND: now also R37.2, R38.2, R39.2, SW3.5, SW3.6, SW3.7, SW3.8, SW4.3 (C), SW5.3 (C), SW6.3 (C)
- net MOT_FAULT: no longer R2.1
- new net: R48.1, SW5.2 (B)
- new net: D4.1 (K), R37.1
- new net: R49.1, SW6.2 (B)
- new net: D6.1 (K), R39.1
- new net: R47.1, SW4.2 (B)
- new net: D5.1 (K), R38.1
- new net BUTT1: R47.2
- new net BUTT2: R48.2
- new net BUTT3: R49.2
- new net DIP_1: R40.2, SW3.1
- new net DIP_2: R41.2, SW3.2
- new net DIP_3: R42.2, SW3.3
- new net DIP_4: R43.2, SW3.4
- new net LED_BLUE: D5.2 (A)
- new net LED_GREEN: D6.2 (A)
- new net LED_RED: D4.2 (A)
- new net MOT1_FAULT: R2.1
- new net MOT2_FAULT: R44.1
- new net MOT3_FAULT: R45.1
- new net MOT4_FAULT: R46.1
Other:
- note added: "Basic LEDs"
- note added: "DIP Switches"
- note added: "Debug buttons"
- note added: "Faults pulled high; fault if low"
- note added: "Neopixel indicator"
- note removed: "Shared pullup for all motor faults (OR)"
- note removed: "Software Indicators"
- moved on the sheet: R2, U1A, U1B

Commit message: Revise following review 1
Parts:
- added J8: ENC1, symbol Connector:Screw_Terminal_01x04
- added J9: ENC2, symbol Connector:Screw_Terminal_01x04
Connections:
- net +5V: now also J8.3 (Pin_3), J9.3 (Pin_3)
- net BUTT1: now also U2.89 (PG4)
- net BUTT2: now also U2.88 (PG3)
- net BUTT3: now also U2.87 (PG2)
- net DIP_1: now also U2.93 (PG8)
- net DIP_2: now also U2.92 (PG7)
- net DIP_3: now also U2.91 (PG6)
- net DIP_4: now also U2.90 (PG5)
- net GND: now also J8.4 (Pin_4), J9.4 (Pin_4)
- net ENC1_A: now reaches U2.34 (PA0)
- net ENC1_A: now also J8.1 (Pin_1)
- net ENC1_B: now reaches U2.35 (PA1)
- net ENC1_B: now also J8.2 (Pin_2)
- net ENC2_A: now reaches U2.96 (PC6)
- net ENC2_A: now also J9.1 (Pin_1)
- net ENC2_B: now reaches U2.97 (PC7)
- net ENC2_B: now also J9.2 (Pin_2)
- net MOT_FAULT: no longer names the net of U2.123 (PD7)
- no-connect marks 102 -> 90
Other:
- note added: "Encoders"
- note added: "TIM2"
- note added: "TIM3"
- note added: "TODO: check A vs B"
