File: sram_external.kicad_sch (KiCad schematic)
At the start: 3 parts, among them U10 23LC1024-I/ST

Commit message: Revise following review 1
Parts:
- U10: footprint ul_23LC1024-I-ST:TSSOP8_MC_MCH -> TSSOP8_MC_MCH
Changed lines of the file:
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@@
 			)
 		)
-		(property "Footprint" "ul_23LC1024-I-ST:TSSOP8_MC_MCH"
+		(property "Footprint" "TSSOP8_MC_MCH"
 			(at 95.25 95.25 0)
 			(effects
